File: SWREG.sch (KiCad schematic (older format))
At the start: 7 parts

Commit message: initiial layout
Other:
- note added: "MANUALLY ADD VCC TO PIN 11 IN LAYOUT"
Changed lines of the file:
@@
 $Descr A4 11693 8268
 encoding utf-8
-Sheet 2 5
+Sheet 2 6
 Title ""
 Date ""
@@
 	4150 2000 5350 2000
 Connection ~ 5350 2000
+Text Notes 3100 1250 0    60   ~ 0
+MANUALLY ADD VCC TO PIN 11 IN LAYOUT
 $EndSCHEMATC
