File: motor2.sch (KiCad schematic (older format))
At the start: 4 parts, among them U3 DRV8839

Commit message: initiial layout
Parts:
- removed C5: 100uF, Capacitors_SMD:c_elec_5x5.3, symbol CP1
- removed C6, C7: 0.1uF, Capacitors_SMD:C_0603, symbol C
- removed U3: DRV8839, customFootprints:SOIC-12-DRV8839, symbol DRV8839
- added C10, C9: 0.1uF, Capacitors_SMD:C_0603, symbol C
- added C8: 100uF, Capacitors_SMD:c_elec_5x5.3, symbol CP1
- added U4: DRV8839, customFootprints:SOIC-12-DRV8839, symbol DRV8839
Connections:
- net EN1: now also U4.9 (EN1)
- net EN2: now also U4.7 (EN2)
- net GND: now also C10.2, C8.2, C9.2, U4.13 (PAD), U4.5 (GND), U4.6 (GND)
- net IN1: now also U4.10 (IN1)
- net IN2: now also U4.8 (IN2)
- net O1: now also U4.3 (OUT1)
- net O2: now also U4.4 (OUT2)
- net VCC: now also C10.1, U4.12 (VCC)
- net VMOT: now also C8.1, C9.1, U4.1 (VM), U4.2 (VM)
- net ~SLEEP: now also U4.11 (SLEEP)
Changed lines of the file:
@@
 $Descr A4 11693 8268
 encoding utf-8
-Sheet 5 6
+Sheet 6 6
 Title ""
 Date ""
@@
 GND
 $Comp
-L DRV8839 U3
-U 1 1 5947EB43
+L DRV8839 U4
+U 1 1 594742BA
 P 3600 1750
-AR Path="/5947EB43" Ref="U3"  Part="1"
-AR Path="/5947EA89/5947EB43" Ref="U3"  Part="1"
-F 0 "U3" H 3600 2200 60  0000 C CNN
+AR Path="/5947EA89/594742BA" Ref="U4"  Part="1"
+AR Path="/594A6AB6/594742BA" Ref="U4"  Part="1"
+AR Path="/594742BA" Ref="U4"  Part="1"
+F 0 "U4" H 3600 2200 60  0000 C CNN
 F 1 "DRV8839" H 3600 2100 60  0000 C CNN
 F 2 "customFootprints:SOIC-12-DRV8839" H 3150 1750 60  0001 C CNN
@@
 Connection ~ 3100 2000
 $Comp
-L C C7
-U 1 1 59481069
+L C C10
+U 1 1 594742BB
 P 5100 1700
-F 0 "C7" H 5125 1800 50  0000 L CNN
+AR Path="/5947EA89/594742BB" Ref="C10"  Part="1"
+AR Path="/594A6AB6/594742BB" Ref="C10"  Part="1"
+F 0 "C10" H 5125 1800 50  0000 L CNN
 F 1 "0.1uF" H 5125 1600 50  0000 L CNN
 F 2 "Capacitors_SMD:C_0603" H 5138 1550 50  0001 C CNN
@@
 	5100 2300 5100 1850
 $Comp
-L C C6
-U 1 1 594810E1
+L C C9
+U 1 1 594742BC
 P 2150 1700
-F 0 "C6" H 2175 1800 50  0000 L CNN
+AR Path="/5947EA89/594742BC" Ref="C9"  Part="1"
+AR Path="/594A6AB6/594742BC" Ref="C9"  Part="1"
+F 0 "C9" H 2175 1800 50  0000 L CNN
 F 1 "0.1uF" H 2175 1600 50  0000 L CNN
 F 2 "Capacitors_SMD:C_0603" H 2188 1550 50  0001 C CNN
@@
 $EndComp
 $Comp
-L CP1 C5
-U 1 1 5948133C
+L CP1 C8
+U 1 1 594742BD
 P 1950 1700
-F 0 "C5" H 1975 1800 50  0000 L CNN
+AR Path="/5947EA89/594742BD" Ref="C8"  Part="1"
+AR Path="/594A6AB6/594742BD" Ref="C8"  Part="1"
+F 0 "C8" H 1975 1800 50  0000 L CNN
 F 1 "100uF" H 1975 1600 50  0000 L CNN
 F 2 "Capacitors_SMD:c_elec_5x5.3" H 1950 1700 50  0001 C CNN
