File: tencm.sch (KiCad schematic (older format))
At the start: 13 parts, among them J1 CONN_01X03, J2 CONN_01X03, J3 CONN_01X03, P1 FIO_HEADER, SW1 PTS810

Commit message: initiial layout
Parts:
- added F1: MINISMDC200F-2, Resistors_SMD:R_1812_HandSoldering, symbol FUSE
- added P3, P4: 1984617, Terminal_Blocks:TerminalBlock_Pheonix_PT-3.5mm_2pol, symbol CONN_01X02
- added PCELL1, PCELL2: S2B-PH-K-S(LF)(SN), Connectors_JST_PH:Connectors_JST_S2B-PH-K, symbol CONN_01X02
- added RS1: 0.1, MF_Passives:MF_Passives-R1206, symbol R
- added U5: INA219BIDCNT, w_smd_trans:sot23-8, symbol INA219BIDCNT
- J1, J2, J3: footprint (none) -> Pin_Headers:Pin_Header_Straight_1x03
- P2: renamed from P?; footprint (none) -> Pin_Headers:Pin_Header_Straight_1x01
- W3, W5: footprint (none) -> Measurement_Points:Measurement_Point_Round-TH_Small
- WBATT1: renamed from WBATT; footprint (none) -> Measurement_Points:Measurement_Point_Round-TH_Small
- WGND1: renamed from WGND; footprint (none) -> Measurement_Points:Measurement_Point_Round-TH_Small
- gave numbers to parts that had none: 3
Connections:
- net 5V0 is gone; now on net 5v0: U2.1 (IN), U2.3 (EN)
- net D9 is gone; now on net GYRO_INT: P1.10 (D9)
- net 3v3_SEL: now also U5.4 (VSS)
- net GND: now also PCELL2.2 (P2), U5.3 (GND), U5.7 (A0), U5.8 (A1)
- net GYRO_INT: no longer P1.3 (D2)
- net GYRO_RST: now also P1.22 (A5); no longer P1.7 (D6)
- net SCL: now also P1.4 (D3), U5.5 (SCL); no longer P1.6 (D5)
- net SDA: now also P1.3 (D2), U5.6 (SDA); no longer P1.5 (D4)
- net VBATT: now also RS1.1, U5.2 (IN-)
- net M1I2: now reaches P1.8 (D7)
- net D8: now reaches P1.9 (D8)
- net D10 renamed M2I1
- net D11 renamed M2I2
- net D14: no longer names the net of P1.13 (D14)
- new net: F1.1, PCELL1.1 (P1)
- new net: PCELL1.2 (P2), PCELL2.1 (P1)
- new net: F1.2, RS1.2, U5.1 (IN+)
- new net M1E: P1.6 (D5)
- new net M1I1: P1.5 (D4)
- new net M2E: P1.7 (D6)
- new net motor/O1: P3.1 (P1)
- new net motor/O2: P3.2 (P2)
- new net motor2/O1: P4.1 (P1)
- new net motor2/O2: P4.2 (P2)
Other:
- note added: "I'm out of non-SPI GPIO pins,\nexcept for dual-use ADC+GPIO pins\nA5 is also Arduino pin 23"
- note added: "PIN 1 POSITIVE"
- note added: "Resistor: Avoid net conflict.\nIt'dn't've been an issue if\npin I/O states were known"
- note added: "TODO:\n[X] BNO055 sym and fp\n[X] Motor driver added\n[X] BNO055 added\n[X] Battery input\n[X] 3v3 source select\n[X] motor power source select\n[X] polyfuses"
- note removed: "Resistor: Avoid net conflict.\nIt'dn't've been an issue\nexcept for damage to Fio"
- note removed: "TODO:\n[X] BNO055 sym and fp\n[X] Motor driver added\n[X] BNO055 added\n[ ] Battery input\n[X] 3v3 source select\n[X] motor power source select\n[ ] polyfuses"
